Commit message: Update optical_offset_x property value

File: urdf/zed_macro.urdf.xacro (robot description, xacro)
@@ -90,5 +90,5 @@
       <xacro:property name="screw_offset_x" value="0.0" />
       <xacro:property name="screw_offset_z" value="-0.016" />
-      <xacro:property name="optical_offset_x" value="-0.005" />
+      <xacro:property name="optical_offset_x" value="0.01" />
       <xacro:property name="mono" value="false" />
       <xacro:property name="mat" value="0.25 0.25 0.25 1.0" />
